Commit message: 042022

File: src/diffbot_description/diffbot_description/urdf/diffbot_description.urdf.xacro (robot description, xacro)
@@ -9,6 +9,6 @@
   <xacro:property name="base_height" value="0.05" />
   <xacro:property name="wheel_mass" value="0.3" /> <!-- arbitrary value for wheel mass -->
-  <xacro:property name="wheel_len" value="0.020" />
-  <xacro:property name="wheel_radius" value="0.015" />
+  <xacro:property name="wheel_len" value="0.57" />
+  <xacro:property name="wheel_radius" value="0.1" />
   <xacro:property name="caster_wheel_mass" value="0.1" /> <!-- arbitrary value for caster wheel mass -->
   <xacro:property name="caster_wheel_radius" value="0.015" />

Commit message: Add files via upload
2022/04/22 diffbot upload

File: src/diffbot_description/diffbot_description/urdf/diffbot_description.urdf.xacro (robot description, xacro)
@@ -9,6 +9,6 @@
   <xacro:property name="base_height" value="0.05" />
   <xacro:property name="wheel_mass" value="0.3" /> <!-- arbitrary value for wheel mass -->
-  <xacro:property name="wheel_len" value="0.57" />
-  <xacro:property name="wheel_radius" value="0.1" />
+  <xacro:property name="wheel_len" value="0.05" />
+  <xacro:property name="wheel_radius" value="0.01" />
   <xacro:property name="caster_wheel_mass" value="0.1" /> <!-- arbitrary value for caster wheel mass -->
   <xacro:property name="caster_wheel_radius" value="0.015" />
